File: elec/layout/default/laser-monitor.kicad_pcb (KiCad board)
At the start: 2 copper layers, 225.7 x 100.8 mm, 0 parts

Commit message: Done
Parts:
- added C1: 50V 100nF X7R ±10% 0603 Multilayer Ceramic Capacitors MLCC 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, lib:C0603, F.Cu at (154.9, 94.7)
- added C2: 50V 100nF X7R ±10% 0603 Multilayer Ceramic Capacitors MLCC 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, lib:C0603, F.Cu at (152.1, 94.5)
- added R1: 62.5mW Thick Film Resistors 50V ±100ppm/℃ ±1% 5.1kΩ 0402 Ch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, lib:R0402, F.Cu at (158.8, 76.7)
- added R10: 62.5mW Thick Film Resistors 50V ±800ppm/℃ ±1% 0Ω 0402 Chip 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, lib:R0402, F.Cu at (147.1, 93.7)
- added R2: 62.5mW Thick Film Resistors 50V ±100ppm/℃ ±1% 5.1kΩ 0402 Ch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, lib:R0402, F.Cu at (158.8, 73.9)
- added R3: 62.5mW Thick Film Resistors 50V ±100ppm/℃ ±1% 10kΩ 0402 Chi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, lib:R0402, F.Cu at (152.1, 89.7)
- added R4: 62.5mW Thick Film Resistors 50V ±100ppm/℃ ±1% 249kΩ 0402 Ch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, lib:R0402, F.Cu at (149.1, 91.7)
- added R5: 62.5mW Thick Film Resistors 50V ±800ppm/℃ ±1% 0Ω 0402 Chip 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, lib:R0402, F.Cu at (150.6, 88.1)
- added R6: 62.5mW Thick Film Resistors 50V ±800ppm/℃ ±1% 0Ω 0402 Chip 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, lib:R0402, F.Cu at (149.4, 88.1)
- added R7: 62.5mW Thick Film Resistors 50V ±800ppm/℃ ±1% 0Ω 0402 Chip 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, lib:R0402, F.Cu at (146.3, 86.9)
- added R8: 62.5mW Thick Film Resistors 50V ±800ppm/℃ ±1% 0Ω 0402 Chip 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, lib:R0402, F.Cu at (146.3, 89.2)
- added R9: 62.5mW Thick Film Resistors 50V ±800ppm/℃ ±1% 0Ω 0402 Chip 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, lib:R0402, F.Cu at (147.1, 96.3)
- added U1: ?, lib:USB-C-SMD_KH-TYPE-C-16P, F.Cu at (164.3, 74.4)
- added U2: ?, lib:LFCSP-8_L3.0-W3.0-P0.50-BL-EP-1, F.Cu at (152.1, 91.9)
- added U3: ?, lib:RES-ADJ-TH_3296W, F.Cu at (146.6, 77.5)
- added U4: ?, lib:SENSOR-SMD_L4.4-W3.9, F.Cu at (142.5, 87.1)
- added U5: ?, lib:LED-TH_BD5.8-P2.54-FD, F.Cu at (142.5, 95.0)
- added U6: ?, lib:BNC-TH_DOSIN-801-0051, F.Cu at (162.6, 91.9)
Routing:
- net usb-gnd: track 0.00 -> 83.0 mm, vias 0 -> 2
- net vcc: track 0.00 -> 37.1 mm, vias 0 -> 2
- net trim_pot-b_t: track 0.00 -> 11.3 mm
- net trim_pot-a_t: track 0.00 -> 10.8 mm
- net amp-b: track 0.00 -> 10.5 mm
- net out: track 0.00 -> 9.07 mm
- net fb: track 0.00 -> 5.13 mm
- net photodiode1-a_t: track 0.00 -> 4.60 mm
- net photodiode2-b_t: track 0.00 -> 4.06 mm
- net photodiode2-a_t: track 0.00 -> 4.06 mm
- net photodiode1-b_t: track 0.00 -> 3.87 mm
- net cc2: track 0.00 -> 3.84 mm
- net cc1: track 0.00 -> 3.33 mm
- net dp: track 0.00 -> 2.92 mm
- net dm: track 0.00 -> 2.90 mm
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Other:
- board size 225.7 x 100.8 mm -> 35 x 35 mm
